File: Backplane/Power.sch (KiCad schematic (older format))
At the start: 33 parts, among them J2 FAN, J3 PWR, Q1 IRFML8244, Q2 AOD4189, Q3 AOD4189, Q4 MMBT3906, Q5 MMBT3904, Q6 MMBT3904

Commit message: Finished to send to fab
Parts:
- removed J2: FAN, conn-100mil:CONN-100MIL-M-1x3, symbol CONN-100MIL-M-1x3
- removed J3: PWR, conn-100mil:CONN-100MIL-M-1x3, symbol CONN-100MIL-M-1x3
- added J2: FAN, conn-100mil:CONN-100MIL-M-1x3-SHROUD, symbol CONN-100MIL-M-1x3-SHROUD
- added J3: POWER, conn-100mil:CONN-100MIL-M-1x3, symbol CONN-100MIL-M-1x4
Connections:
- net 12V: now also J2.2
- net GND: now also J3.1, J3.4
- net at RT1.1: now also J3.2, J3.3
- net at D1.2, Q1.3: now also J2.1, J2.3
Changed lines of the file:
@@
 3SBCS
 Connection ~ 6400 4900
-$Comp
-L CONN-100MIL-M-1x3 J3
-U 1 1 54D6F85F
-P 750 4000
-F 0 "J3" H 750 4200 50  0000 C CNN
-F 1 "PWR" H 750 4100 50  0000 C CNN
-F 2 "conn-100mil:CONN-100MIL-M-1x3" H 750 4000 50  0001 C CNN
-F 3 "" H 750 4000 50  0000 C CNN
-F 4 "J8" H 750 4000 50  0001 C CNN "OldReference"
-	1    750  4000
-	-1   0    0    -1
-$EndComp
 Wire Wire Line
 	800  4000 900  4000
 Wire Wire Line
-	900  4000 900  4300
-Wire Wire Line
-	900  4200 800  4200
-Connection ~ 900  4200
+	900  4000 900  4400
 $Comp
 L GND #PWR0209
 U 1 1 54D7002D
-P 900 4300
-F 0 "#PWR0209" H 900 4300 30  0001 C CNN
-F 1 "GND" H 900 4230 30  0001 C CNN
-F 2 "" H 900 4300 60  0000 C CNN
-F 3 "" H 900 4300 60  0000 C CNN
-F 4 "#PWR0207" H 900 4300 50  0001 C CNN "OldReference"
-	1    900  4300
+P 900 4400
+F 0 "#PWR0209" H 900 4400 30  0001 C CNN
+F 1 "GND" H 900 4330 30  0001 C CNN
+F 2 "" H 900 4400 60  0000 C CNN
+F 3 "" H 900 4400 60  0000 C CNN
+F 4 "#PWR0207" H 900 4400 50  0001 C CNN "OldReference"
+	1    900  4400
 	1    0    0    -1
 $EndComp
 Wire Wire Line
 	5250 1900 6000 1900
-$Comp
-L CONN-100MIL-M-1x3 J2
-U 1 1 54D81D58
-P 9750 1200
-F 0 "J2" H 9750 1400 50  0000 C CNN
-F 1 "FAN" H 9750 1300 50  0000 C CNN
-F 2 "conn-100mil:CONN-100MIL-M-1x3" H 9750 1200 50  0001 C CNN
-F 3 "" H 9750 1200 50  0000 C CNN
-F 4 "J10" H 9750 1200 50  0001 C CNN "OldReference"
-	1    9750 1200
-	1    0    0    -1
-$EndComp
 Wire Wire Line
 	9500 1200 9700 1200
@@
 3V3
 Wire Wire Line
-	10100 2400 7200 2400
+	7200 2400 10100 2400
 Wire Wire Line
 	6000 2400 3700 2400
@@
 	7850 2350 7850 2400
 Connection ~ 7850 2400
+$Comp
+L CONN-100MIL-M-1x4 J3
+U 1 1 54EB5D17
+P 750 4000
+F 0 "J3" H 750 4200 50  0000 C CNN
+F 1 "POWER" H 750 4100 50  0000 C CNN
+F 2 "conn-100mil:CONN-100MIL-M-1x3" H 750 4000 50  0001 C CNN
+F 3 "" H 750 4000 50  0000 C CNN
+	1    750  4000
+	-1   0    0    -1
+$EndComp
+Wire Wire Line
+	800  4300 900  4300
+Connection ~ 900  4300
+Wire Wire Line
+	850  4100 850  4200
+Wire Wire Line
+	850  4200 800  4200
+Connection ~ 850  4100
+$Comp
+L CONN-100MIL-M-1x3-SHROUD J2
+U 1 1 54EB8F00
+P 9750 1200
+F 0 "J2" H 9750 1400 50  0000 C CNN
+F 1 "FAN" H 9750 1300 50  0000 C CNN
+F 2 "conn-100mil:CONN-100MIL-M-1x3-SHROUD" H 9750 1200 50  0001 C CNN
+F 3 "" H 9750 1200 50  0000 C CNN
+	1    9750 1200
+	1    0    0    -1
+$EndComp
 $EndSCHEMATC
