File: Frontend/Atten1.sch (KiCad schematic (older format))
At the start: 64 parts

Commit message: Frontend schematic ready to go to layout
Parts:
- removed C? (x2): 100n, IPC7351-Nominal:CAPC1608X55, symbol C-0603
- removed C?: 5p6, symbol C
- removed C?: 2p7, IPC7351-Nominal:CAPC1005X55, symbol C-0402
- removed C?: 1p, IPC7351-Nominal:CAPC1005X55, symbol C-0402
- removed C? (x2): 2p2, IPC7351-Nominal:CAPC1005X55, symbol C-0402
- removed CV?: SGC3S100, symbol CVAR
- removed J?: INPUT, conn-linx:CONN-CONSMA001, symbol CONN-CONSMA001
- removed L?: 68n, IPC7351-Nominal:INDC1005X60, symbol L-0402
- removed R? (x3): 33, IPC7351-Nominal:RESC1005X40, symbol R-0402
- removed R?: 68, IPC7351-Nominal:RESC1608X50, symbol R-0603
- removed R? (x3): 332k, IPC7351-Nominal:RESC2012X50, symbol R-0805
- removed R?: 75, IPC7351-Nominal:RESC1608X50, symbol R-0603
- removed R?: 3k3, IPC7351-Nominal:RESC1608X50, symbol R-0603
- removed R? (x3): 470, IPC7351-Nominal:RESC1005X40, symbol R-0402
- removed R?: 68, IPC7351-Nominal:RESC1005X40, symbol R-0402
- removed R?: 143, IPC7351-Nominal:RESC1005X40, symbol R-0402
- removed R?: 270, IPC7351-Nominal:RESC1005X40, symbol R-0402
- removed R?: 680, IPC7351-Nominal:RESC1005X40, symbol R-0402
- removed R?: 150, IPC7351-Nominal:RESC1005X40, symbol R-0402
- removed R? (x2): 100, IPC7351-Nominal:RESC1005X40, symbol R-0402
- removed R? (x2): 402, IPC7351-Nominal:RESC1005X40, symbol R-0402
- removed R? (x2): 49R9, IPC7351-Nominal:RESC1005X40, symbol R-0402
- removed R? (x4): 200, IPC7351-Nominal:RESC3216X60, symbol R-1206
- removed SW? (x2): SPDT, symbol SPDT
- removed U? (x2): ADA4817-1ACPZ, manuf:ANALOG-LFCSP_VD-8, symbol ADA4817-1ACPZ
- removed U? (x2): AD8003ACPZ, IPC7351-Nominal:QFN50P400X400X80-25, symbol AD8003ACPZ
- removed U?: VCA821IDGST, IPC7351-Nominal:SOP50P490X110-10, symbol VCA821IDGST
- removed U?: LMH6552SD, IPC7351-Nominal:PSON50P300X250X80-9, symbol LMH6552SD
- added C? (x9): 100n, IPC7351-Nominal:CAPC1608X55, symbol C-0603
- added C?: 10p 1kV, IPC7351-Nominal:CAPC3216X70, symbol C-1206
- added C?: 4p7 1kV, IPC7351-Nominal:CAPC3216X70, symbol C-1206
- added C?: 120p, IPC7351-Nominal:CAPC2012X70, symbol C-0805
- added C?: 10p, IPC7351-Nominal:CAPC2012X70, symbol C-0805
- added CV? (x2): 30p, symbol CVAR
- added R? (x4): 200, IPC7351-Nominal:RESC3216X60, symbol R-1206
- added R?: 33, IPC7351-Nominal:RESC1005X40, symbol R-0402
- added R?: 3k3, IPC7351-Nominal:RESC1608X50, symbol R-0603
- added R? (x3): 332k, IPC7351-Nominal:RESC2012X50, symbol R-0805
- added R?: 75, IPC7351-Nominal:RESC1608X50, symbol R-0603
- added R?: 10M, IPC7351-Nominal:RESC2012X50, symbol R-0805
- added R? (x2): 357k, IPC7351-Nominal:RESC2012X50, symbol R-0805
- added R?: 348k, IPC7351-Nominal:RESC2012X50, symbol R-0805
- added R?: 165, IPC7351-Nominal:RESC2012X50, symbol R-0805
- added R?: 35R7, IPC7351-Nominal:RESC2012X50, symbol R-0805
- added R? (x4): 30, IPC7351-Nominal:RESC2012X50, symbol R-0805
- added R?: 200, IPC7351-Nominal:RESC2012X50, symbol R-0805
- added R? (x2): 443, IPC7351-Nominal:RESC1608X50, symbol R-0603
- added R? (x2): 120, IPC7351-Nominal:RESC1608X50, symbol R-0603
- added R? (x2): 49r9, IPC7351-Nominal:RESC1608X50, symbol R-0603
- added R?: 120, IPC7351-Nominal:RESC2012X50, symbol R-0805
- added R? (x2): 300, IPC7351-Nominal:RESC1608X50, symbol R-0603
- added R? (x2): 64R9, IPC7351-Nominal:RESC1608X50, symbol R-0603
- added R?: 432, IPC7351-Nominal:RESC1608X50, symbol R-0603
- added SW? (x6): DPDT, symbol DPDT
- added U? (x2): ADA4817-1ACPZ, manuf:ANALOG-LFCSP_VD-8, symbol ADA4817-1ACPZ
- added U? (x4): AD8003ACPZ, IPC7351-Nominal:QFN50P400X400X80-25, symbol AD8003ACPZ
- added U? (x2): LMH6552SD, IPC7351-Nominal:PSON50P300X250X80-9, symbol LMH6552SD
- CV?: value 44p -> 30p
- D?: BOM (none) -> DIST DIGIKEY 568-1624-1-ND; Manuf (none) -> Value
- GDT?: BOM (none) -> DIST DIGIKEY 2051-40-SM-RPLFCT-ND
- R? (x2): value 390k -> 357k
- R?: value 332k -> 348k
- R? (x2): value 3M -> 523k
- R?: value 3M -> 536k
Connections:
- net labels added: INPUT, VOCM, VO_N, VO_P
- net labels removed: OUT+, OUT-, VCOM, VGAIN
- wire segments 153 -> 230
Other:
- note added: "+15dB"
- note added: "+6dB"
- note added: "-15dB"
- note added: "-30dB"
- note added: "-6dB"
- moved on the sheet: CV?, R?
