File: Frontend/Channel.sch (KiCad schematic (older format))
At the start: 98 parts, among them K4 HE3600, K5 EE2-5NU, K6 HE3600, U15 MC33078DGK, U23 MCP9700T-E/TT, U24 ADA4817-1ACPZ, U25 MAX4567EEE, U26 MAX4567EEE, U27 AD8003ACPZ, U28 MAX4567EEE, U29 LMH6552SD, U30 MC33078DGK

Commit message: Route PCB
Parts:
- removed R114, R124: 49r9, IPC7351-Nominal:RESC1608X50, symbol R-0603
- added R114, R124: 49R9, IPC7351-Nominal:RESC1005X40, symbol R-0402
- renumbered U30 to U15
Connections:
- net -5: now also U24.5 (V-); no longer U24.9 (PAD)
- net GND: now also U24.9 (PAD); no longer U24.5 (V-)
- net VO_N: now also R124.1
- net VO_P: now also R114.1
- net at R113.1, U29.4 (OUT+): now also R114.2
- net at R123.1, U29.5 (OUT-): now also R124.2
- net at R116.1, U27.2 (FB): now also R112.2
- net at U27.8 (OUT): no longer R112.2

Commit message: More layout work
Parts:
- removed C92: 33u/16, IPC7351-Nominal:CAPMP7343X310, symbol C-TANT-7343-31
- added C115, C117: TBD, IPC7351-Nominal:CAPC1005X55, symbol C-0402
- added R141, R143: TBD, IPC7351-Nominal:RESC1005X40, symbol R-0402
Connections:
- net GND: now also C115.2, C117.2
- net at R117.1, R118.2, U27.16 (IN-): now also R141.1
- net at R120.1, R121.2, U27.21 (IN-): now also R143.1
- new net: C117.1, R143.2
- new net: C115.1, R141.2
Other:
- note added: "This capacitor is only\npresent in channel 2."

Commit message: Schematic touchups
Connections:
- no-connect marks 1 -> 2

Commit message: Route #IRQ and #PERST
Changed lines of the file:
@@
 LIBS:Altera
 LIBS:conn-te
+LIBS:Vishay
+LIBS:semi-trans-OnSemi
 LIBS:frontend-cache
 EELAYER 25 0
@@
 AR Path="/54E51D33/5552E99B" Ref="#C1"  Part="1"
 AR Path="/552E2A83/5552E99B" Ref="C16"  Part="1"
-F 0 "#C1" H 1200 8750 50  0000 C CNN
+F 0 "#C1" H 1200 8750 50  0001 C CNN
 F 1 "33u/16" H 1200 8650 50  0000 C CNN
 F 2 "IPC7351-Nominal:CAPMP7343X310" H 900 8700 50  0001 C CNN

Commit message: Reannotate schematic/PCB
Parts:
- renumbered C77 to C1, C115 to C10, C117 to C11, C86 to C12, C87 to C13, C88 to C14, C89 to C15, C90 to C16, C91 to C17, C93 to C19, C78 to C2, C94 to C20, C95 to C21, C96 to C22, C97 to C23, C98 to C24, C99 to C25, C100 to C26, C101 to C27, C102 to C28, C103 to C29, C79 to C3, C104 to C30, C105 to C31, C106 to C32, C107 to C33, C108 to C34, C109 to C35, C110 to C36, C111 to C37, C112 to C38, C80 to C4, C81 to C5, C82 to C6, C83 to C7, C84 to C8, C85 to C9, CV5 to CV1, CV6 to CV2, CV7 to CV3, CV8 to CV4, D5 to D1, D6 to D2, D7 to D3, GDT2 to GDT1, K4 to K1, K5 to K2, K6 to K3, R86 to R1, R95 to R10, R96 to R11, R97 to R12, R98 to R13, R99 to R14, R100 to R15, R101 to R16, R102 to R17, R103 to R18, R104 to R19, R87 to R2, R105 to R20, R106 to R21, R107 to R22, R108 to R23, R109 to R24, R110 to R25, R111 to R26, R112 to R27, R113 to R28, R114 to R29, R88 to R3, R115 to R30, R116 to R31, R117 to R32, R118 to R33, R119 to R34, R120 to R35, R121 to R36, R141 to R37, R143 to R38, R122 to R39, R89 to R4, R123 to R40, R124 to R41, R125 to R42, R126 to R43, R127 to R44, R90 to R5, R91 to R6, R92 to R7, R93 to R8, R94 to R9, U23 to U1, U24 to U2, U25 to U3, U28 to U4, U26 to U5, U27 to U6, U29 to U7, U15 to U8

Commit message: Add bypass capacitor around AC coupling capacitors
Parts:
- added C18: 1n 2kV, IPC7351-Nominal:CAPC4520X168, symbol C-1808
Connections:
- net at C4.1, D1.3, K1.P1A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: now also C18.1
- net at C4.2, K1.P1B, R2.1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: now also C18.2
Other:
- moved on the sheet: C3, C4, K1A, R2

Commit message: Reannotate after adding parts
Parts:
- renumbered C9 to C10, C10 to C11, C11 to C12, C12 to C13, C13 to C14, C14 to C15, C15 to C16, C16 to C17, C17 to C18, C19 to C20, C20 to C21, C21 to C22, C22 to C23, C23 to C24, C24 to C25, C25 to C26, C26 to C27, C27 to C28, C28 to C29, C29 to C30, C30 to C31, C31 to C32, C32 to C33, C33 to C34, C34 to C35, C35 to C36, C36 to C37, C37 to C38, C38 to C39, C18 to C4, C4 to C5, C5 to C6, C6 to C7, C7 to C8, C8 to C9
