File: Frontend/Channel.sch (KiCad schematic (older format))
At the start: 101 parts, among them K1 HE3600, K2 EE2-5NU, K3 HE3600, U1 MCP9700T-E/TT, U2 ADA4817-1ACPZ, U3 MAX4567EEE, U4 MAX4567EEE, U5 MAX4567EEE, U6 AD8003ACPZ, U7 LMH6552SD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

Commit message: Schematic cleanup
Other:
- moved on the sheet: C31, C39, U8B, U8C

Commit message: Cleanup offset compensation system
Parts:
- removed C10: 100n, IPC7351-Nominal:CAPC1608X55, symbol C-0603
- added R67: 20k, IPC7351-Nominal:RESC1005X40, symbol R-0402
- R23: value 150 -> 10k; BOM RES SMD 150 0.5% [0402] -> RES SMD 10k 1% [0402]
Connections:
- net GND: now also U2.4 (IN+)
- net at R23.1: now also R27.1, R28.2, U7.1 (IN-); no longer U2.4 (IN+)
- net at R39.1, R40.2, U7.8 (IN+): now also R67.1
- new net +2.5: R67.2

Commit message: Even more layout tweaks
Parts:
- added TP11, TP13: S2, conn-test:TEST-SMD-SMALL, symbol TESTPOINT
- added TP4: BUFFER, conn-test:TEST-SMD-SMALL, symbol TESTPOINT
- added TP6: S1, conn-test:TEST-SMD-SMALL, symbol TESTPOINT
Connections:
- net at R30.1, U2.7 (OUT), U3.8 (NC1): now also TP4.1
- net at U4.13 (COM2), U6.4 (IN+): now also TP13.1
- net at U3.5 (COM1), U5.10 (NC2), U5.2 (NO1): now also TP6.1
- net at U4.10 (NC2), U4.2 (NO1), U5.13 (COM2): now also TP11.1
Changed lines of the file:
@@
 $EndComp
 Wire Wire Line
-	12700 2000 12700 4300
+	12700 1950 12700 4300
 Wire Wire Line
 	9400 2650 9400 2550
@@
 	11050 6050 11100 6050
 Connection ~ 11400 6050
+$Comp
+L TESTPOINT TP4
+U 1 1 55632DAB
+P 12700 1950
+AR Path="/54E51D33/55632DAB" Ref="TP4"  Part="1"
+AR Path="/552E2A83/55632DAB" Ref="TP5"  Part="1"
+F 0 "TP5" H 12850 2100 50  0000 C CNN
+F 1 "BUFFER" H 12850 2000 50  0000 C CNN
+F 2 "conn-test:TEST-SMD-SMALL" H 12700 1950 50  0001 C CNN
+F 3 "" H 12700 1950 50  0000 C CNN
+	1    12700 1950
+	1    0    0    -1
+$EndComp
+Connection ~ 12700 2000
+$Comp
+L TESTPOINT TP6
+U 1 1 55634827
+P 2000 5200
+AR Path="/54E51D33/55634827" Ref="TP6"  Part="1"
+AR Path="/552E2A83/55634827" Ref="TP7"  Part="1"
+F 0 "TP7" H 2150 5350 50  0000 C CNN
+F 1 "S1" H 2150 5250 50  0000 C CNN
+F 2 "conn-test:TEST-SMD-SMALL" H 2000 5200 50  0001 C CNN
+F 3 "" H 2000 5200 50  0000 C CNN
+	1    2000 5200
+	1    0    0    -1
+$EndComp
+Wire Wire Line
+	2000 5200 2000 5300
+Connection ~ 2000 5300
+$Comp
+L TESTPOINT TP11
+U 1 1 55636805
+P 5200 5300
+AR Path="/54E51D33/55636805" Ref="TP11"  Part="1"
+AR Path="/552E2A83/55636805" Ref="TP12"  Part="1"
+F 0 "TP12" H 5350 5450 50  0000 C CNN
+F 1 "S2" H 5350 5350 50  0000 C CNN
+F 2 "conn-test:TEST-SMD-SMALL" H 5200 5300 50  0001 C CNN
+F 3 "" H 5200 5300 50  0000 C CNN
+	1    5200 5300
+	1    0    0    -1
+$EndComp
+Wire Wire Line
+	5200 5300 5200 5400
+Connection ~ 5200 5400
+$Comp
+L TESTPOINT TP13
+U 1 1 55638366
+P 8500 5200
+AR Path="/54E51D33/55638366" Ref="TP13"  Part="1"
+AR Path="/552E2A83/55638366" Ref="TP14"  Part="1"
+F 0 "TP14" H 8650 5350 50  0000 C CNN
+F 1 "S2" H 8650 5250 50  0000 C CNN
+F 2 "conn-test:TEST-SMD-SMALL" H 8500 5200 50  0001 C CNN
+F 3 "" H 8500 5200 50  0000 C CNN
+	1    8500 5200
+	1    0    0    -1
+$EndComp
+Wire Wire Line
+	8500 5200 8500 5300
+Connection ~ 8500 5300
 $EndSCHEMATC

Commit message: Fix final gain stage resistors
Parts:
- R27, R39: value 150 -> 220; BOM RES SMD 150 0.5% [0402] -> RES SMD 220 0.5% [0402]
Changed lines of the file:
@@
 AR Path="/54E51D33/554FADE0" Ref="R27"  Part="1"
 AR Path="/552E2A83/554FADE0" Ref="R71"  Part="1"
-F 1 "150" V 11100 5400 50  0000 C CNN
 F 0 "R27" V 11000 5400 50  0000 C CNN
+F 1 "220" V 11100 5400 50  0000 C CNN
 F 2 "IPC7351-Nominal:RESC1005X40" H 11200 5400 50  0001 C CNN
 F 3 "" H 11200 5450 60  0000 C CNN
 F 4 "Value" H 11200 5400 60  0001 C CNN "Manuf"
-F 5 "RES SMD 150 0.5% [0402]" H 11950 5950 60  0001 C CNN "BOM"
+F 5 "RES SMD 220 0.5% [0402]" H 11950 5950 60  0001 C CNN "BOM"
 	1    11200 5400
 	0    1    1    0
@@
 AR Path="/54E51D33/554FB1EA" Ref="R39"  Part="1"
 AR Path="/552E2A83/554FB1EA" Ref="R83"  Part="1"
-F 1 "150" V 11100 6500 50  0000 C CNN
 F 0 "R39" V 11000 6500 50  0000 C CNN
+F 1 "220" V 11100 6500 50  0000 C CNN
 F 2 "IPC7351-Nominal:RESC1005X40" H 11200 6500 50  0001 C CNN
 F 3 "" H 11200 6550 60  0000 C CNN
 F 4 "Value" H 11200 6500 60  0001 C CNN "Manuf"
-F 5 "RES SMD 150 0.5% [0402]" H 11950 7050 60  0001 C CNN "BOM"
+F 5 "RES SMD 220 0.5% [0402]" H 11950 7050 60  0001 C CNN "BOM"
 	1    11200 6500
 	0    1    1    0

Commit message: More routing adjustments
Parts:
- removed C3, C7: 4p7 1kV, IPC7351-Nominal:CAPC3216X70, symbol C-1206
- added C3, C7: 4p7 1kV, smd-non-ipc:CAPC2828X260, symbol C-1111
- C5: BOM EF6223-ND -> DIST DIGIKEY EF6223-ND
- C9: BOM CAP MLCC 100pF C0G 50V 5% [0805] -> CAP MLCC 120p C0G 50V 10% [0805]
- R1, R2: value 75 -> 64R9; BOM RES SMD 75 1% [0603] -> RES SMD 64R9 1% [0402]
- R10: value 536k -> 523k; BOM RES SMD 536k 1% [0805] -> RES SMD 523k 1% [0805]
- R20: BOM RES SMD 3k3 5% [0402] -> RES SMD 3k3 1% [0402]
- R24, R26: value 348k -> 357k; BOM RES SMD 348k 1% [0805] -> RES SMD 357k 1% [0805]
- R27, R39: BOM RES SMD 220 0.5% [0402] -> RES SMD 220 1% [0402]
- R28, R31, R40, R43: value 443 -> 442; BOM RES SMD 443 0.5% [0402] -> RES SMD 442 1% [0402]
- R30: BOM RES SMD 165 0.5% [0402] -> RES SMD 165 1% [0402]
- R32, R35: BOM RES SMD 64R9 0.5% [0402] -> RES SMD 64R9 1% [0402]
- R33, R36: BOM RES SMD 300 0.5% [0402] -> RES SMD 300 1% [0402]
- R34: BOM RES SMD 35R7 0.5% [0402] -> RES SMD 35R7 1% [0402]
- R4: value 33 -> 35R7; BOM RES SMD 33 1% [0402] -> RES SMD 35R7 1% [0402]
- R42: BOM RES SMD 91k 1% [0402] -> RES SMD 120k 1% [0402]
- R44: BOM RES SMD 13k 1% [0402] -> RES SMD 30k 1% [0402]
- U7: BOM IC TI LMH6552D -> #IC TI LMH6552D
- U7: BOM DIST DIGIKEY LMH6552SD/NOPBCT-ND -> #IC TI LMH6552D
Connections:
- net at C8.1, K2.P1A, R13.1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: now also C7.2
- net at C9.1, CV3.1, K2.P2A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: now also C7.1
- net at C6.1, K2.P2CO, R5.2: now also C3.2
- net at R2.2: now also C3.1
