File: Frontend/Channel.sch (KiCad schematic (older format))
At the start: 105 parts, among them K1 HE3600, K2 EE2-5NU, K3 HE3600, U1 MCP9700T-E/TT, U2 ADA4817-1ACPZ, U3 MAX4567EEE, U4 MAX4567EEE, U5 MAX4567EEE, U6 AD8003ACPZ, U7 LMH6552SD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

Commit message: Finally finish the final layout finally
Parts:
- removed R20: 3k3, IPC7351-Nominal:RESC1005X40, symbol R-0402
- C13: BOM CAP MLCC 100pF C0G 50V 5% [0603] -> CAP MLCC 100n ≥X5R 25V 20% [0603]
- C31, C39: BOM CAP MLCC 100n ≥X5R 16V 20% [0603] -> CAP MLCC 100n ≥X5R 25V 20% [0603]
- C9: value 120p -> 100p; BOM CAP MLCC 120p C0G 50V 10% [0805] -> CAP MLCC 100p C0G 50V 10% [0805]
- R10, R8, R9: value 523k -> 5M23; BOM RES SMD 523k 1% [0805] -> RES SMD 5M23 1% [0805]
Connections:
- net GUARD is gone; now on net GND: D1.1, D1.2
