File: Frontend/LevelShifters.sch (KiCad schematic (older format))
At the start: 55 parts, among them U11 MC33078DGK, U12 MC33078DGK, U13 MC33078DGK, U14 MC33078DGK

Commit message: Work more on routing
Parts:
- added TP2: V1C1, conn-test:TEST-SMD-SMALL, symbol TESTPOINT
- added TP3: V1C2, conn-test:TEST-SMD-SMALL, symbol TESTPOINT
- added TP4: V2C1, conn-test:TEST-SMD-SMALL, symbol TESTPOINT
- added TP5: V2C2, conn-test:TEST-SMD-SMALL, symbol TESTPOINT
- added TP6: V3C1, conn-test:TEST-SMD-SMALL, symbol TESTPOINT
- added TP7: V3C2, conn-test:TEST-SMD-SMALL, symbol TESTPOINT
Connections:
- net VOS1_CH1_OUT: now also TP2.1
- net VOS1_CH2_OUT: now also TP3.1
- net VOS2_CH1_OUT: now also TP4.1
- net VOS2_CH2_OUT: now also TP5.1
- net VOS3_CH1_OUT: now also TP6.1
- net VOS3_CH2_OUT: now also TP7.1

Commit message: Schematic touchups
Parts:
- C48, C49: BOM CAP MLCC 10n ≥X7R 10V 20% [0402] -> CAP MLCC 10n ≥X7R 16V 20% [0402]
- C50, C51, C52, C53, C54: BOM CAP MLCC 100pF C0G 50V 5% [0603] -> CAP MLCC 100n ≥X7R 25V 20% [0603]
Other:
- note added: "Level shifters are also low-pass filters, due to the\nrelatively high noise of the DAC at frequency above 1 kHz.\n\nfc ~~= 230 Hz\nSetting time to 99.9%: 5.2 ms"
- note removed: "fc ~~= 230 Hz\nSetting time to 99.9%: 5.2 ms"
- moved on the sheet: C50, C55, C56, C57, C58, C59, C60, C61, C62, C63, C64, R59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

Commit message: Reannotate schematic/PCB
Parts:
- renumbered C60 to C100, C61 to C101, C62 to C102, C63 to C103, C64 to C104, C48 to C88, C49 to C89, C50 to C90, C51 to C91, C52 to C92, C53 to C93, C54 to C94, C55 to C95, C56 to C96, C57 to C97, C58 to C98, C59 to C99, R49 to R111, R50 to R112, R51 to R113, R52 to R114, R53 to R115, R54 to R116, R55 to R117, R56 to R118, R57 to R119, R58 to R120, R59 to R121, R60 to R122, R61 to R123, R62 to R124, R63 to R125, R64 to R126, R65 to R127, R66 to R128, R67 to R129, R68 to R130, R69 to R131, R70 to R132, R71 to R133, R72 to R134, R73 to R135, R74 to R136, R75 to R137, R76 to R138, R77 to R139, R78 to R140, R79 to R141, R80 to R142, R81 to R143, R82 to R144, U11 to U19, U12 to U20, U13 to U21, U14 to U22

Commit message: Reannotate after adding parts
Parts:
- renumbered C98 to C100, C99 to C101, C100 to C102, C101 to C103, C102 to C104, C103 to C105, C104 to C106, C88 to C90, C89 to C91, C90 to C92, C91 to C93, C92 to C94, C93 to C95, C94 to C96, C95 to C97, C96 to C98, C97 to C99
Changed lines of the file:
@@
 P 5450 3400
 AR Path="/552B011F/55501BFF" Ref="C?"  Part="1"
-AR Path="/552B011F/5550176D/55501BFF" Ref="C91"  Part="1"
-F 0 "C91" V 5200 3400 50  0000 C CNN
+AR Path="/552B011F/5550176D/55501BFF" Ref="C93"  Part="1"
+F 0 "C93" V 5200 3400 50  0000 C CNN
 F 1 "100n" V 5300 3400 50  0000 C CNN
 F 2 "IPC7351-Nominal:CAPC1608X55" H 5450 3400 50  0001 C CNN
@@
 P 8500 3400
 AR Path="/552B011F/55501C1E" Ref="C?"  Part="1"
-AR Path="/552B011F/5550176D/55501C1E" Ref="C92"  Part="1"
-F 0 "C92" V 8250 3400 50  0000 C CNN
+AR Path="/552B011F/5550176D/55501C1E" Ref="C94"  Part="1"
+F 0 "C94" V 8250 3400 50  0000 C CNN
 F 1 "100n" V 8350 3400 50  0000 C CNN
 F 2 "IPC7351-Nominal:CAPC1608X55" H 8500 3400 50  0001 C CNN
@@
 P 5450 5000
 AR Path="/552B011F/55501C69" Ref="C?"  Part="1"
-AR Path="/552B011F/5550176D/55501C69" Ref="C93"  Part="1"
-F 0 "C93" V 5200 5000 50  0000 C CNN
+AR Path="/552B011F/5550176D/55501C69" Ref="C95"  Part="1"
+F 0 "C95" V 5200 5000 50  0000 C CNN
 F 1 "100n" V 5300 5000 50  0000 C CNN
 F 2 "IPC7351-Nominal:CAPC1608X55" H 5450 5000 50  0001 C CNN
@@
 P 2200 2500
 AR Path="/552B011F/55501C74" Ref="C?"  Part="1"
-AR Path="/552B011F/5550176D/55501C74" Ref="C90"  Part="1"
-F 0 "C90" V 1950 2500 50  0000 C CNN
+AR Path="/552B011F/5550176D/55501C74" Ref="C92"  Part="1"
+F 0 "C92" V 1950 2500 50  0000 C CNN
 F 1 "100n" V 2050 2500 50  0000 C CNN
 F 2 "IPC7351-Nominal:CAPC1608X55" H 2200 2500 50  0001 C CNN
@@
 AR Path="/54E51D33/55501DC3" Ref="C?"  Part="1"
 AR Path="/552B011F/55501DC3" Ref="C?"  Part="1"
-AR Path="/552B011F/5550176D/55501DC3" Ref="C88"  Part="1"
-F 0 "C88" V 5200 1800 50  0000 C CNN
+AR Path="/552B011F/5550176D/55501DC3" Ref="C90"  Part="1"
+F 0 "C90" V 5200 1800 50  0000 C CNN
 F 1 "10n" V 5300 1800 50  0000 C CNN
 F 2 "IPC7351-Nominal:CAPC1005X55" H 5450 1800 50  0001 C CNN
@@
 AR Path="/54E51D33/55501E06" Ref="C?"  Part="1"
 AR Path="/552B011F/55501E06" Ref="C?"  Part="1"
-AR Path="/552B011F/5550176D/55501E06" Ref="C89"  Part="1"
-F 0 "C89" V 8100 1800 50  0000 C CNN
+AR Path="/552B011F/5550176D/55501E06" Ref="C91"  Part="1"
+F 0 "C91" V 8100 1800 50  0000 C CNN
 F 1 "10n" V 8200 1800 50  0000 C CNN
 F 2 "IPC7351-Nominal:CAPC1005X55" H 8350 1800 50  0001 C CNN
@@
 P 8350 5000
 AR Path="/552B011F/55501E56" Ref="C?"  Part="1"
-AR Path="/552B011F/5550176D/55501E56" Ref="C94"  Part="1"
-F 0 "C94" V 8100 5000 50  0000 C CNN
+AR Path="/552B011F/5550176D/55501E56" Ref="C96"  Part="1"
+F 0 "C96" V 8100 5000 50  0000 C CNN
 F 1 "100n" V 8200 5000 50  0000 C CNN
 F 2 "IPC7351-Nominal:CAPC1608X55" H 8350 5000 50  0001 C CNN
@@
 AR Path="/54E51D33/555044AB" Ref="C?"  Part="1"
 AR Path="/552B011F/555044AB" Ref="C?"  Part="1"
-AR Path="/552B011F/5550176D/555044AB" Ref="C96"  Part="1"
-F 0 "C96" H 2150 6950 50  0000 C CNN
+AR Path="/552B011F/5550176D/555044AB" Ref="C98"  Part="1"
+F 0 "C98" H 2150 6950 50  0000 C CNN
 F 1 "100n" H 2150 6850 50  0000 C CNN
 F 2 "IPC7351-Nominal:CAPC1608X55" H 1900 6900 50  0001 C CNN
@@
 AR Path="/54E51D33/555044B4" Ref="C?"  Part="1"
 AR Path="/552B011F/555044B4" Ref="C?"  Part="1"
-AR Path="/552B011F/5550176D/555044B4" Ref="C101"  Part="1"
-F 0 "C101" H 2150 7350 50  0000 C CNN
+AR Path="/552B011F/5550176D/555044B4" Ref="C103"  Part="1"
+F 0 "C103" H 2150 7350 50  0000 C CNN
 F 1 "100n" H 2150 7250 50  0000 C CNN
 F 2 "IPC7351-Nominal:CAPC1608X55" H 1900 7300 50  0001 C CNN
@@
 AR Path="/54E51D33/555044BD" Ref="C?"  Part="1"
 AR Path="/552B011F/555044BD" Ref="C?"  Part="1"
-AR Path="/552B011F/5550176D/555044BD" Ref="C102"  Part="1"
-F 0 "C102" H 2950 7350 50  0000 C CNN
+AR Path="/552B011F/5550176D/555044BD" Ref="C104"  Part="1"
+F 0 "C104" H 2950 7350 50  0000 C CNN
 F 1 "100n" H 2950 7250 50  0000 C CNN
 F 2 "IPC7351-Nominal:CAPC1608X55" H 2700 7300 50  0001 C CNN
@@
 AR Path="/54E51D33/555044C6" Ref="C?"  Part="1"
 AR Path="/552B011F/555044C6" Ref="C?"  Part="1"
-AR Path="/552B011F/5550176D/555044C6" Ref="C97"  Part="1"
-F 0 "C97" H 2950 6950 50  0000 C CNN
+AR Path="/552B011F/5550176D/555044C6" Ref="C99"  Part="1"
+F 0 "C99" H 2950 6950 50  0000 C CNN
 F 1 "100n" H 2950 6850 50  0000 C CNN
 F 2 "IPC7351-Nominal:CAPC1608X55" H 2700 6900 50  0001 C CNN
@@
 AR Path="/54E51D33/555044CF" Ref="C?"  Part="1"
 AR Path="/552B011F/555044CF" Ref="C?"  Part="1"
-AR Path="/552B011F/5550176D/555044CF" Ref="C98"  Part="1"
-F 0 "C98" H 3750 6950 50  0000 C CNN
+AR Path="/552B011F/5550176D/555044CF" Ref="C100"  Part="1"
+F 0 "C100" H 3750 6950 50  0000 C CNN
 F 1 "100n" H 3750 6850 50  0000 C CNN
 F 2 "IPC7351-Nominal:CAPC1608X55" H 3500 6900 50  0001 C CNN
@@
 AR Path="/54E51D33/555044D8" Ref="C?"  Part="1"
 AR Path="/552B011F/555044D8" Ref="C?"  Part="1"
-AR Path="/552B011F/5550176D/555044D8" Ref="C103"  Part="1"
-F 0 "C103" H 3750 7350 50  0000 C CNN
+AR Path="/552B011F/5550176D/555044D8" Ref="C105"  Part="1"
+F 0 "C105" H 3750 7350 50  0000 C CNN
 F 1 "100n" H 3750 7250 50  0000 C CNN
 F 2 "IPC7351-Nominal:CAPC1608X55" H 3500 7300 50  0001 C CNN
@@
 AR Path="/54E51D33/555044E1" Ref="C?"  Part="1"
 AR Path="/552B011F/555044E1" Ref="C?"  Part="1"
-AR Path="/552B011F/5550176D/555044E1" Ref="C104"  Part="1"
-F 0 "C104" H 4550 7350 50  0000 C CNN
+AR Path="/552B011F/5550176D/555044E1" Ref="C106"  Part="1"
+F 0 "C106" H 4550 7350 50  0000 C CNN
 F 1 "100n" H 4550 7250 50  0000 C CNN
 F 2 "IPC7351-Nominal:CAPC1608X55" H 4300 7300 50  0001 C CNN
@@
 AR Path="/54E51D33/555044EA" Ref="C?"  Part="1"
 AR Path="/552B011F/555044EA" Ref="C?"  Part="1"
-AR Path="/552B011F/5550176D/555044EA" Ref="C99"  Part="1"
-F 0 "C99" H 4550 6950 50  0000 C CNN
+AR Path="/552B011F/5550176D/555044EA" Ref="C101"  Part="1"
+F 0 "C101" H 4550 6950 50  0000 C CNN
 F 1 "100n" H 4550 6850 50  0000 C CNN
 F 2 "IPC7351-Nominal:CAPC1608X55" H 4300 6900 50  0001 C CNN
@@
 P 900 6900
 AR Path="/552B011F/555578F2" Ref="C?"  Part="1"
-AR Path="/552B011F/5550176D/555578F2" Ref="C95"  Part="1"
-F 0 "C95" H 1150 6950 50  0000 C CNN
+AR Path="/552B011F/5550176D/555578F2" Ref="C97"  Part="1"
+F 0 "C97" H 1150 6950 50  0000 C CNN
 F 1 "15u/16" H 1150 6850 50  0000 C CNN
 F 2 "IPC7351-Nominal:CAPMP3528X210" H 900 6900 50  0001 C CNN
@@
 P 900 7300
 AR Path="/552B011F/55557975" Ref="C?"  Part="1"
-AR Path="/552B011F/5550176D/55557975" Ref="C100"  Part="1"
-F 0 "C100" H 1150 7350 50  0000 C CNN
+AR Path="/552B011F/5550176D/55557975" Ref="C102"  Part="1"
+F 0 "C102" H 1150 7350 50  0000 C CNN
 F 1 "15u/16" H 1150 7250 50  0000 C CNN
 F 2 "IPC7351-Nominal:CAPMP3528X210" H 900 7300 50  0001 C CNN
