File: Frontend/Power.sch (KiCad schematic (older format))
At the start: 26 parts, among them J11 APWR, U19 LM317S, U20 L78M05CDT, U21 MCP1700T-3302E/TT, U22 MC79M05CDT

Commit message: Route PCB
Parts:
- removed MP1: 217-36CTE6, symbol HEATSINK-NO-CONN
- added MP1: 217-36CTE6, symbol HEATSINK-CONN
- R83: footprint (none) -> manuf:KOASPEER-MOS-2W
- U21: footprint (none) -> smd-semi:SOT-23
Connections:
- net labels added: VRHS
- wire segments 54 -> 56
Changed lines of the file:
@@
 $EndComp
 $Comp
-L GND #PWR0200
+L GND #PWR0202
 U 1 1 552FAC91
 P 3800 4300
-F 0 "#PWR0200" H 3800 4300 30  0001 C CNN
+F 0 "#PWR0202" H 3800 4300 30  0001 C CNN
 F 1 "GND" H 3800 4230 30  0001 C CNN
 F 2 "" H 3800 4300 60  0000 C CNN
@@
 $EndComp
 $Comp
-L GND #PWR0201
+L GND #PWR0203
 U 1 1 552FB1F9
 P 4400 4300
-F 0 "#PWR0201" H 4400 4300 30  0001 C CNN
+F 0 "#PWR0203" H 4400 4300 30  0001 C CNN
 F 1 "GND" H 4400 4230 30  0001 C CNN
 F 2 "" H 4400 4300 60  0000 C CNN
@@
 $EndComp
 $Comp
-L GND #PWR0202
+L GND #PWR0204
 U 1 1 552FB410
 P 4800 4300
-F 0 "#PWR0202" H 4800 4300 30  0001 C CNN
+F 0 "#PWR0204" H 4800 4300 30  0001 C CNN
 F 1 "GND" H 4800 4230 30  0001 C CNN
 F 2 "" H 4800 4300 60  0000 C CNN
@@
 $EndComp
 $Comp
-L GND #PWR0203
+L GND #PWR0205
 U 1 1 552FBBCC
 P 5350 4300
-F 0 "#PWR0203" H 5350 4300 30  0001 C CNN
+F 0 "#PWR0205" H 5350 4300 30  0001 C CNN
 F 1 "GND" H 5350 4230 30  0001 C CNN
 F 2 "" H 5350 4300 60  0000 C CNN
@@
 $EndComp
 $Comp
-L GND #PWR0204
+L GND #PWR0206
 U 1 1 552FBE04
 P 5800 4300
-F 0 "#PWR0204" H 5800 4300 30  0001 C CNN
+F 0 "#PWR0206" H 5800 4300 30  0001 C CNN
 F 1 "GND" H 5800 4230 30  0001 C CNN
 F 2 "" H 5800 4300 60  0000 C CNN
@@
 $EndComp
 $Comp
-L -5 #PWR0205
+L -5 #PWR0207
 U 1 1 552FBF15
 P 5800 3850
-F 0 "#PWR0205" H 5800 3800 30  0001 C CNN
+F 0 "#PWR0207" H 5800 3800 30  0001 C CNN
 F 1 "-5" H 5800 3750 50  0000 C CNN
 F 2 "" H 5800 3850 60  0000 C CNN
@@
 $EndComp
 $Comp
-L GND #PWR0206
+L GND #PWR0208
 U 1 1 552FD87A
 P 6200 2350
-F 0 "#PWR0206" H 6200 2350 30  0001 C CNN
+F 0 "#PWR0208" H 6200 2350 30  0001 C CNN
 F 1 "GND" H 6200 2280 30  0001 C CNN
 F 2 "" H 6200 2350 60  0000 C CNN
@@
 $EndComp
 $Comp
-L +12 #PWR0207
+L +12 #PWR0209
 U 1 1 5530425A
 P 3600 1900
-F 0 "#PWR0207" H 3600 1950 30  0001 C CNN
+F 0 "#PWR0209" H 3600 1950 30  0001 C CNN
 F 1 "+12" H 3600 2000 50  0000 C CNN
 F 2 "" H 3600 1900 60  0000 C CNN
@@
 Connection ~ 5800 2400
 $Comp
-L GND #PWR0208
+L GND #PWR0210
 U 1 1 5547D09D
 P 5800 2800
-F 0 "#PWR0208" H 5800 2800 30  0001 C CNN
+F 0 "#PWR0210" H 5800 2800 30  0001 C CNN
 F 1 "GND" H 5800 2730 30  0001 C CNN
 F 2 "" H 5800 2800 60  0000 C CNN
@@
 	5800 2800 5800 2700
 Connection ~ 5800 2000
-$Comp
-L HEATSINK-NO-CONN MP1
-U 1 1 5547D192
-P 5350 1600
-F 0 "MP1" H 5350 2050 50  0000 C CNN
-F 1 "217-36CTE6" H 5350 1950 50  0000 C CNN
-F 2 "" H 5350 1600 60  0000 C CNN
-F 3 "" H 5350 1600 60  0000 C CNN
-	1    5350 1600
-	1    0    0    -1
-$EndComp
 $Comp
 L R R83
@@
 F 0 "R83" V 4000 2000 50  0000 C CNN
 F 1 "15 2W" V 4100 2000 50  0000 C CNN
-F 2 "" H 4200 2050 60  0000 C CNN
+F 2 "manuf:KOASPEER-MOS-2W" H 4200 2050 60  0001 C CNN
 F 3 "" H 4200 2050 60  0000 C CNN
 	1    4200 2000
@@
 Connection ~ 4750 2000
 $Comp
-L GND #PWR0209
+L GND #PWR0211
 U 1 1 55480232
 P 4750 2400
-F 0 "#PWR0209" H 4750 2400 30  0001 C CNN
+F 0 "#PWR0211" H 4750 2400 30  0001 C CNN
 F 1 "GND" H 4750 2330 30  0001 C CNN
 F 2 "" H 4750 2400 60  0000 C CNN
@@
 	5800 3200 5800 3300
 $Comp
-L +5 #PWR0210
+L +5 #PWR0212
 U 1 1 55480B1F
 P 5900 3150
-F 0 "#PWR0210" H 5900 3200 30  0001 C CNN
+F 0 "#PWR0212" H 5900 3200 30  0001 C CNN
 F 1 "+5" H 5900 3250 50  0000 C CNN
 F 2 "" H 5900 3150 60  0000 C CNN
@@
 Connection ~ 5800 3200
 $Comp
-L GND #PWR0211
+L GND #PWR0213
 U 1 1 55480BB8
 P 5350 3550
-F 0 "#PWR0211" H 5350 3550 30  0001 C CNN
+F 0 "#PWR0213" H 5350 3550 30  0001 C CNN
 F 1 "GND" H 5350 3480 30  0001 C CNN
 F 2 "" H 5350 3550 60  0000 C CNN
@@
 	5350 3550 5350 3500
 $Comp
-L GND #PWR0212
+L GND #PWR0214
 U 1 1 55480C51
 P 5800 3550
-F 0 "#PWR0212" H 5800 3550 30  0001 C CNN
+F 0 "#PWR0214" H 5800 3550 30  0001 C CNN
 F 1 "GND" H 5800 3480 30  0001 C CNN
 F 2 "" H 5800 3550 60  0000 C CNN
@@
 	4800 3200 4800 3300
 $Comp
-L GND #PWR0213
+L GND #PWR0215
 U 1 1 55480DAB
 P 4800 3550
-F 0 "#PWR0213" H 4800 3550 30  0001 C CNN
+F 0 "#PWR0215" H 4800 3550 30  0001 C CNN
 F 1 "GND" H 4800 3480 30  0001 C CNN
 F 2 "" H 4800 3550 60  0000 C CNN
@@
 Connection ~ 4800 3200
 $Comp
-L +8 #PWR0214
+L +8 #PWR0216
 U 1 1 55480F09
 P 3700 3150
-F 0 "#PWR0214" H 3700 3200 30  0001 C CNN
+F 0 "#PWR0216" H 3700 3200 30  0001 C CNN
 F 1 "+8" H 3700 3250 50  0000 C CNN
 F 2 "" H 3700 3150 60  0000 C CNN
@@
 Connection ~ 4400 3200
 $Comp
-L GND #PWR0215
+L GND #PWR0217
 U 1 1 55481C45
 P 4400 3550
-F 0 "#PWR0215" H 4400 3550 30  0001 C CNN
+F 0 "#PWR0217" H 4400 3550 30  0001 C CNN
 F 1 "GND" H 4400 3480 30  0001 C CNN
 F 2 "" H 4400 3550 60  0000 C CNN
@@
 Connection ~ 3800 3200
 $Comp
-L GND #PWR0216
+L GND #PWR0218
 U 1 1 55481E79
 P 3800 3550
-F 0 "#PWR0216" H 3800 3550 30  0001 C CNN
+F 0 "#PWR0218" H 3800 3550 30  0001 C CNN
 F 1 "GND" H 3800 3480 30  0001 C CNN
 F 2 "" H 3800 3550 60  0000 C CNN
@@
 	3800 3550 3800 3500
 $Comp
-L -8 #PWR0217
+L -8 #PWR0219
 U 1 1 55482517
 P 3700 3850
-F 0 "#PWR0217" H 3700 3800 30  0001 C CNN
+F 0 "#PWR0219" H 3700 3800 30  0001 C CNN
 F 1 "-8" H 3700 3750 50  0000 C CNN
 F 2 "" H 3700 3850 60  0000 C CNN
@@
 	3800 3900 3800 4000
 $Comp
-L GND #PWR0218
+L GND #PWR0220
 U 1 1 55483EF7
 P 2600 3650
-F 0 "#PWR0218" H 2600 3650 30  0001 C CNN
+F 0 "#PWR0220" H 2600 3650 30  0001 C CNN
 F 1 "GND" H 2600 3580 30  0001 C CNN
 F 2 "" H 2600 3650 60  0000 C CNN
@@
 F 0 "U21" H 6750 3500 50  0000 C CNN
 F 1 "MCP1700T-3302E/TT" H 6750 3400 50  0000 C CNN
-F 2 "" H 6750 3250 60  0000 C CNN
+F 2 "smd-semi:SOT-23" H 6750 3250 60  0001 C CNN
 F 3 "" H 6750 3250 60  0000 C CNN
 F 4 "IC MICROCHIP MCP1700T-3302E/TT" H 7250 4000 60  0001 C CNN "BOM"
@@
 Connection ~ 5900 3200
 $Comp
-L GND #PWR0219
+L GND #PWR0221
 U 1 1 555465A7
 P 6750 3550
-F 0 "#PWR0219" H 6750 3550 30  0001 C CNN
+F 0 "#PWR0221" H 6750 3550 30  0001 C CNN
 F 1 "GND" H 6750 3480 30  0001 C CNN
 F 2 "" H 6750 3550 60  0000 C CNN
@@
 Connection ~ 6200 3200
 $Comp
-L GND #PWR0220
+L GND #PWR0222
 U 1 1 55548553
 P 6200 3550
-F 0 "#PWR0220" H 6200 3550 30  0001 C CNN
+F 0 "#PWR0222" H 6200 3550 30  0001 C CNN
 F 1 "GND" H 6200 3480 30  0001 C CNN
 F 2 "" H 6200 3550 60  0000 C CNN
@@
 	7200 3200 7200 3300
 $Comp
-L GND #PWR0221
+L GND #PWR0223
 U 1 1 5554875C
 P 7200 3550
-F 0 "#PWR0221" H 7200 3550 30  0001 C CNN
+F 0 "#PWR0223" H 7200 3550 30  0001 C CNN
 F 1 "GND" H 7200 3480 30  0001 C CNN
 F 2 "" H 7200 3550 60  0000 C CNN
@@
 +3.3A
 Connection ~ 7200 3200
+$Comp
+L HEATSINK-CONN MP1
+U 1 1 55503A38
+P 5350 1550
+F 0 "MP1" H 5350 2000 50  0000 C CNN
+F 1 "217-36CTE6" H 5350 1900 50  0000 C CNN
+F 2 "" H 5350 1550 60  0000 C CNN
+F 3 "" H 5350 1550 60  0000 C CNN
+	1    5350 1550
+	1    0    0    -1
+$EndComp
+Wire Wire Line
+	5350 1650 5750 1650
+Wire Wire Line
+	5750 1650 5750 2000
+Connection ~ 5750 2000
+Text Label 5750 1650 2    60   ~ 0
+VRHS
 $EndSCHEMATC

Commit message: Work more on routing
Parts:
- MP1: footprint (none) -> manuf:LAIRD-BMI-S-203
Changed lines of the file:
@@
 $EndComp
 $Comp
-L GND #PWR0202
+L GND #PWR0214
 U 1 1 552FAC91
 P 3800 4300
-F 0 "#PWR0202" H 3800 4300 30  0001 C CNN
+F 0 "#PWR0214" H 3800 4300 30  0001 C CNN
 F 1 "GND" H 3800 4230 30  0001 C CNN
 F 2 "" H 3800 4300 60  0000 C CNN
@@
 $EndComp
 $Comp
-L GND #PWR0203
+L GND #PWR0215
 U 1 1 552FB1F9
 P 4400 4300
-F 0 "#PWR0203" H 4400 4300 30  0001 C CNN
+F 0 "#PWR0215" H 4400 4300 30  0001 C CNN
 F 1 "GND" H 4400 4230 30  0001 C CNN
 F 2 "" H 4400 4300 60  0000 C CNN
@@
 $EndComp
 $Comp
-L GND #PWR0204
+L GND #PWR0216
 U 1 1 552FB410
 P 4800 4300
-F 0 "#PWR0204" H 4800 4300 30  0001 C CNN
+F 0 "#PWR0216" H 4800 4300 30  0001 C CNN
 F 1 "GND" H 4800 4230 30  0001 C CNN
 F 2 "" H 4800 4300 60  0000 C CNN
@@
 $EndComp
 $Comp
-L GND #PWR0205
+L GND #PWR0217
 U 1 1 552FBBCC
 P 5350 4300
-F 0 "#PWR0205" H 5350 4300 30  0001 C CNN
+F 0 "#PWR0217" H 5350 4300 30  0001 C CNN
 F 1 "GND" H 5350 4230 30  0001 C CNN
 F 2 "" H 5350 4300 60  0000 C CNN
@@
 $EndComp
 $Comp
-L GND #PWR0206
+L GND #PWR0218
 U 1 1 552FBE04
 P 5800 4300
-F 0 "#PWR0206" H 5800 4300 30  0001 C CNN
+F 0 "#PWR0218" H 5800 4300 30  0001 C CNN
 F 1 "GND" H 5800 4230 30  0001 C CNN
 F 2 "" H 5800 4300 60  0000 C CNN
@@
 $EndComp
 $Comp
-L -5 #PWR0207
+L -5 #PWR0219
 U 1 1 552FBF15
 P 5800 3850
-F 0 "#PWR0207" H 5800 3800 30  0001 C CNN
+F 0 "#PWR0219" H 5800 3800 30  0001 C CNN
 F 1 "-5" H 5800 3750 50  0000 C CNN
 F 2 "" H 5800 3850 60  0000 C CNN
@@
 $EndComp
 $Comp
-L GND #PWR0208
+L GND #PWR0220
 U 1 1 552FD87A
 P 6200 2350
-F 0 "#PWR0208" H 6200 2350 30  0001 C CNN
+F 0 "#PWR0220" H 6200 2350 30  0001 C CNN
 F 1 "GND" H 6200 2280 30  0001 C CNN
 F 2 "" H 6200 2350 60  0000 C CNN
@@
 $EndComp
 $Comp
-L +12 #PWR0209
+L +12 #PWR0221
 U 1 1 5530425A
 P 3600 1900
-F 0 "#PWR0209" H 3600 1950 30  0001 C CNN
+F 0 "#PWR0221" H 3600 1950 30  0001 C CNN
 F 1 "+12" H 3600 2000 50  0000 C CNN
 F 2 "" H 3600 1900 60  0000 C CNN
@@
 Connection ~ 5800 2400
 $Comp
-L GND #PWR0210
+L GND #PWR0222
 U 1 1 5547D09D
 P 5800 2800
-F 0 "#PWR0210" H 5800 2800 30  0001 C CNN
+F 0 "#PWR0222" H 5800 2800 30  0001 C CNN
 F 1 "GND" H 5800 2730 30  0001 C CNN
 F 2 "" H 5800 2800 60  0000 C CNN
@@
 Connection ~ 4750 2000
 $Comp
-L GND #PWR0211
+L GND #PWR0223
 U 1 1 55480232
 P 4750 2400
-F 0 "#PWR0211" H 4750 2400 30  0001 C CNN
+F 0 "#PWR0223" H 4750 2400 30  0001 C CNN
 F 1 "GND" H 4750 2330 30  0001 C CNN
 F 2 "" H 4750 2400 60  0000 C CNN
@@
 	5800 3200 5800 3300
 $Comp
-L +5 #PWR0212
+L +5 #PWR0224
 U 1 1 55480B1F
 P 5900 3150
-F 0 "#PWR0212" H 5900 3200 30  0001 C CNN
+F 0 "#PWR0224" H 5900 3200 30  0001 C CNN
 F 1 "+5" H 5900 3250 50  0000 C CNN
 F 2 "" H 5900 3150 60  0000 C CNN
@@
 Connection ~ 5800 3200
 $Comp
-L GND #PWR0213
+L GND #PWR0225
 U 1 1 55480BB8
 P 5350 3550
-F 0 "#PWR0213" H 5350 3550 30  0001 C CNN
+F 0 "#PWR0225" H 5350 3550 30  0001 C CNN
 F 1 "GND" H 5350 3480 30  0001 C CNN
 F 2 "" H 5350 3550 60  0000 C CNN
@@
 	5350 3550 5350 3500
 $Comp
-L GND #PWR0214
+L GND #PWR0226
 U 1 1 55480C51
 P 5800 3550
-F 0 "#PWR0214" H 5800 3550 30  0001 C CNN
+F 0 "#PWR0226" H 5800 3550 30  0001 C CNN
 F 1 "GND" H 5800 3480 30  0001 C CNN
 F 2 "" H 5800 3550 60  0000 C CNN
@@
 	4800 3200 4800 3300
 $Comp
-L GND #PWR0215
+L GND #PWR0227
 U 1 1 55480DAB
 P 4800 3550
-F 0 "#PWR0215" H 4800 3550 30  0001 C CNN
+F 0 "#PWR0227" H 4800 3550 30  0001 C CNN
 F 1 "GND" H 4800 3480 30  0001 C CNN
 F 2 "" H 4800 3550 60  0000 C CNN
@@
 Connection ~ 4800 3200
 $Comp
-L +8 #PWR0216
+L +8 #PWR0228
 U 1 1 55480F09
 P 3700 3150
-F 0 "#PWR0216" H 3700 3200 30  0001 C CNN
+F 0 "#PWR0228" H 3700 3200 30  0001 C CNN
 F 1 "+8" H 3700 3250 50  0000 C CNN
 F 2 "" H 3700 3150 60  0000 C CNN
@@
 Connection ~ 4400 3200
 $Comp
-L GND #PWR0217
+L GND #PWR0229
 U 1 1 55481C45
 P 4400 3550
-F 0 "#PWR0217" H 4400 3550 30  0001 C CNN
+F 0 "#PWR0229" H 4400 3550 30  0001 C CNN
 F 1 "GND" H 4400 3480 30  0001 C CNN
 F 2 "" H 4400 3550 60  0000 C CNN
@@
 Connection ~ 3800 3200
 $Comp
-L GND #PWR0218
+L GND #PWR0230
 U 1 1 55481E79
 P 3800 3550
-F 0 "#PWR0218" H 3800 3550 30  0001 C CNN
+F 0 "#PWR0230" H 3800 3550 30  0001 C CNN
 F 1 "GND" H 3800 3480 30  0001 C CNN
 F 2 "" H 3800 3550 60  0000 C CNN
@@
 	3800 3550 3800 3500
 $Comp
-L -8 #PWR0219
+L -8 #PWR0231
 U 1 1 55482517
 P 3700 3850
-F 0 "#PWR0219" H 3700 3800 30  0001 C CNN
+F 0 "#PWR0231" H 3700 3800 30  0001 C CNN
 F 1 "-8" H 3700 3750 50  0000 C CNN
 F 2 "" H 3700 3850 60  0000 C CNN
@@
 	3800 3900 3800 4000
 $Comp
-L GND #PWR0220
+L GND #PWR0232
 U 1 1 55483EF7
 P 2600 3650
-F 0 "#PWR0220" H 2600 3650 30  0001 C CNN
+F 0 "#PWR0232" H 2600 3650 30  0001 C CNN
 F 1 "GND" H 2600 3580 30  0001 C CNN
 F 2 "" H 2600 3650 60  0000 C CNN
@@
 Connection ~ 5900 3200
 $Comp
-L GND #PWR0221
+L GND #PWR0233
 U 1 1 555465A7
 P 6750 3550
-F 0 "#PWR0221" H 6750 3550 30  0001 C CNN
+F 0 "#PWR0233" H 6750 3550 30  0001 C CNN
 F 1 "GND" H 6750 3480 30  0001 C CNN
 F 2 "" H 6750 3550 60  0000 C CNN
@@
 Connection ~ 6200 3200
 $Comp
-L GND #PWR0222
+L GND #PWR0234
 U 1 1 55548553
 P 6200 3550
-F 0 "#PWR0222" H 6200 3550 30  0001 C CNN
+F 0 "#PWR0234" H 6200 3550 30  0001 C CNN
 F 1 "GND" H 6200 3480 30  0001 C CNN
 F 2 "" H 6200 3550 60  0000 C CNN
@@
 	7200 3200 7200 3300
 $Comp
-L GND #PWR0223
+L GND #PWR0235
 U 1 1 5554875C
 P 7200 3550
-F 0 "#PWR0223" H 7200 3550 30  0001 C CNN
+F 0 "#PWR0235" H 7200 3550 30  0001 C CNN
 F 1 "GND" H 7200 3480 30  0001 C CNN
 F 2 "" H 7200 3550 60  0000 C CNN
@@
 F 0 "MP1" H 5350 2000 50  0000 C CNN
 F 1 "217-36CTE6" H 5350 1900 50  0000 C CNN
-F 2 "" H 5350 1550 60  0000 C CNN
+F 2 "manuf:LAIRD-BMI-S-203" H 5350 1550 60  0001 C CNN
 F 3 "" H 5350 1550 60  0000 C CNN
 	1    5350 1550

Commit message: More layout work
Parts:
- removed C67, C69, C73, C75: 47u, pth-passive:C-ALUM-5mm, symbol C-ALUM-5mm
- removed E5, E7: 120, IPC7351-Nominal:RESC3216X60, symbol BEAD-1206
- removed U21: MCP1700T-3302E/TT, smd-semi:SOT-23, symbol MCP1700T-vv02E/TT
- added C118, C119: 1u, IPC7351-Nominal:CAPC2012X70, symbol C-0805
- added C67, C73: 330u, pth-passive:C-ALUM-8mm, symbol C-ALUM-8mm
- added R148: 100k, IPC7351-Nominal:RESC1608X50, symbol R-0603
- added U16, U17: MCP9700T-E/TT, smd-semi:SOT-23, symbol MCP9700T-E/TT
- added U18: TLV70233DSE, manuf:TEXAS-S-PWSON-N6, symbol TLV702vvDSE
Connections:
- net labels added: +3.3, TEMP_V5, TEMP_VRELAY
- wire segments 56 -> 72
Other:
- moved on the sheet: C71, C72

Commit message: Schematic touchups
Connections:
- net labels added: PWR
- wire segments 72 -> 69
Other:
- note added: "The analog 3.3V rail is enabled by the digital 3.3V rail, so the\nDAC is not powered if separate analog power cable is\ndisconnected. @R148 forms a low-pass filter with the input and\noutput capacitors to prevent injection of noise from the digital rail."
- moved on the sheet: C118, C119, C65, C66, C67, C68, C70, C71, C72, C73, C74, C76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

Commit message: Reannotate schematic/PCB
Parts:
- renumbered C65 to C105, C66 to C106, C118 to C107, C119 to C108, C67 to C109, C68 to C110, C70 to C111, C71 to C112, C72 to C113, C73 to C114, C74 to C115, C76 to C116, D4 to D7, E6 to E5, R83 to R145, R84 to R146, R85 to R147, U19 to U23, U16 to U24, U20 to U25, U18 to U26, U17 to U27, U22 to U28

Commit message: Reannotate after adding parts
Parts:
- renumbered C105 to C107, C106 to C108, C107 to C109, C108 to C110, C109 to C111, C110 to C112, C111 to C113, C112 to C114, C113 to C115, C114 to C116, C115 to C117, C116 to C118
Changed lines of the file:
@@
 $EndComp
 $Comp
-L C-0603 C115
+L C-0603 C117
 U 1 1 552FB081
 P 3300 5200
-F 0 "C115" H 3500 5250 50  0000 C CNN
+F 0 "C117" H 3500 5250 50  0000 C CNN
 F 1 "100n" H 3500 5150 50  0000 C CNN
 F 2 "IPC7351-Nominal:CAPC1608X55" H 3300 5200 50  0001 C CNN
@@
 	2500 2900 3000 2900
 $Comp
-L C-ALUM-5mm C105
+L C-ALUM-5mm C107
 U 1 1 5548016D
 P 3650 3100
-F 0 "C105" H 3850 3150 50  0000 C CNN
+F 0 "C107" H 3850 3150 50  0000 C CNN
 F 1 "47u" H 3850 3050 50  0000 C CNN
 F 2 "pth-passive:C-ALUM-5mm" H 3650 3100 50  0001 C CNN
@@
 $EndComp
 $Comp
-L C-0603 C110
+L C-0603 C112
 U 1 1 55481B7D
 P 3300 4500
-F 0 "C110" H 3500 4550 50  0000 C CNN
+F 0 "C112" H 3500 4550 50  0000 C CNN
 F 1 "100n" H 3500 4450 50  0000 C CNN
 F 2 "IPC7351-Nominal:CAPC1608X55" H 3300 4500 50  0001 C CNN
@@
 Connection ~ 1500 4500
 $Comp
-L C-ALUM-5mm C111
+L C-ALUM-5mm C113
 U 1 1 55556F9E
 P 4700 4500
-F 0 "C111" H 4900 4550 50  0000 C CNN
+F 0 "C113" H 4900 4550 50  0000 C CNN
 F 1 "47u" H 4900 4450 50  0000 C CNN
 F 2 "pth-passive:C-ALUM-5mm" H 4700 4500 50  0001 C CNN
@@
 $EndComp
 $Comp
-L C-ALUM-5mm C116
+L C-ALUM-5mm C118
 U 1 1 55556FF0
 P 4700 5200
-F 0 "C116" H 4900 5150 50  0000 C CNN
+F 0 "C118" H 4900 5150 50  0000 C CNN
 F 1 "47u" H 4900 5250 50  0000 C CNN
 F 2 "pth-passive:C-ALUM-5mm" H 4700 5200 50  0001 C CNN
@@
 $EndComp
 $Comp
-L C-ALUM-5mm C106
+L C-ALUM-5mm C108
 U 1 1 5555707F
 P 5100 3100
-F 0 "C106" H 5300 3150 50  0000 C CNN
+F 0 "C108" H 5300 3150 50  0000 C CNN
 F 1 "47u" H 5300 3050 50  0000 C CNN
 F 2 "pth-passive:C-ALUM-5mm" H 5100 3100 50  0001 C CNN
@@
 	6500 4400 6500 4550
 $Comp
-L C-0805 C112
+L C-0805 C114
 U 1 1 555483A0
 P 5200 4500
-F 0 "C112" H 5400 4550 50  0000 C CNN
+F 0 "C114" H 5400 4550 50  0000 C CNN
 F 1 "1u" H 5400 4450 50  0000 C CNN
 F 2 "IPC7351-Nominal:CAPC2012X70" H 5200 4500 50  0001 C CNN
@@
 	5200 4650 5200 4600
 $Comp
-L C-0805 C113
+L C-0805 C115
 U 1 1 555486B6
 P 6700 4500
-F 0 "C113" H 6900 4550 50  0000 C CNN
+F 0 "C115" H 6900 4550 50  0000 C CNN
 F 1 "1u" H 6900 4450 50  0000 C CNN
 F 2 "IPC7351-Nominal:CAPC2012X70" H 6700 4500 50  0001 C CNN
@@
 	8050 3400 8100 3400
 $Comp
-L C-0805 C107
+L C-0805 C109
 U 1 1 55547120
 P 7700 3300
-AR Path="/552F27A6/55547120" Ref="C107"  Part="1"
+AR Path="/552F27A6/55547120" Ref="C109"  Part="1"
 AR Path="/54E51D33/55547120" Ref="C?"  Part="1"
 AR Path="/552E2A83/55547120" Ref="C?"  Part="1"
-F 0 "C107" H 7900 3350 50  0000 C CNN
+F 0 "C109" H 7900 3350 50  0000 C CNN
 F 1 "1u" H 7900 3250 50  0000 C CNN
 F 2 "IPC7351-Nominal:CAPC2012X70" H 7700 3300 50  0001 C CNN
@@
 	8050 4500 8100 4500
 $Comp
-L C-0805 C108
+L C-0805 C110
 U 1 1 555474C5
 P 7700 4400
-AR Path="/552F27A6/555474C5" Ref="C108"  Part="1"
+AR Path="/552F27A6/555474C5" Ref="C110"  Part="1"
 AR Path="/54E51D33/555474C5" Ref="C?"  Part="1"
 AR Path="/552E2A83/555474C5" Ref="C?"  Part="1"
-F 0 "C108" H 7900 4450 50  0000 C CNN
+F 0 "C110" H 7900 4450 50  0000 C CNN
 F 1 "1u" H 7900 4350 50  0000 C CNN
 F 2 "IPC7351-Nominal:CAPC2012X70" H 7700 4400 50  0001 C CNN
@@
 	9300 4400 9100 4400
 $Comp
-L C-ALUM-8mm C109
+L C-ALUM-8mm C111
 U 1 1 55540904
 P 2700 4500
-F 0 "C109" H 2900 4550 50  0000 C CNN
+F 0 "C111" H 2900 4550 50  0000 C CNN
 F 1 "330u" H 2900 4450 50  0000 C CNN
 F 2 "pth-passive:C-ALUM-8mm" H 2700 4500 50  0001 C CNN
@@
 $EndComp
 $Comp
-L C-ALUM-8mm C114
+L C-ALUM-8mm C116
 U 1 1 5554115A
 P 2700 5200
-F 0 "C114" H 2900 5150 50  0000 C CNN
+F 0 "C116" H 2900 5150 50  0000 C CNN
 F 1 "330u" H 2900 5250 50  0000 C CNN
 F 2 "pth-passive:C-ALUM-8mm" H 2700 5200 50  0001 C CNN
