File: Frontend/frontend.kicad_pcb (KiCad board)
At the start: 4 copper layers, 100 x 100.2 mm, 340 parts, among them J1 SATA, J10 SWD, J11 APWR, J2 BNC, J3 SATA, J6 BNC, J9 PCIEx4 EDGE, K1 HE3600, K2 EE2-5NU, K3 HE3600, K4 HE3600, K5 EE2-5NU, K6 HE3600, Q1 ULN2003AD, U1 MCP9700T-E/TT, U10 ADA4817-1ACPZ, U11 MAX4567EEE, U12 MAX4567EEE, U13 MAX4567EEE, U14 AD8003ACPZ, U15 LMH6552SD, U16 MC33078DGK, U17 MAX5725AAUP, U18 STM32F030C8T, U19 MC33078DGK, U2 ADA4817-1ACPZ, U20 MC33078DGK, U23 LM317S, U24 MCP9700T-E/TT, U25 L78M05CDT, U26 TLV70233DSE, U27 MCP9700T-E/TT, U28 MC79M05CDT, U3 MAX4567EEE, U4 MAX4567EEE, U5 MAX4567EEE, U6 AD8003ACPZ, U7 LMH6552SD, U8 MC33078DGK, U9 MCP9700T-E/TT

Commit message: Finally finish the final layout finally
Parts:
- removed R20, R64: 3k3, IPC7351-Nominal:RESC1005X40
- C48, C9: value 120p -> 100p
- R10, R54: value 536k -> 5M23
- R24, R26, R68, R70: value 348k -> 357k
- R52, R53, R8, R9: value 523k -> 5M23
- moved C43 0.15 mm to (114.5, 83.0)
Connections:
- D1 pad 1: /Channel1/GUARD -> GND
- D1 pad 2: /Channel1/GUARD -> GND
- D4 pad 1: /Channel2/GUARD -> GND
- D4 pad 2: /Channel2/GUARD -> GND
Routing:
- net /Channel2/GUARD: track 86.7 -> 0.00 mm, vias 2 -> 0
- net /Channel1/GUARD: track 86.5 -> 0.00 mm, vias 2 -> 0
- net GND: track 1128.9 -> 1110.1 mm, vias 437 -> 439
- net VRELAY: track 239.4 -> 250.9 mm, vias 8 -> 18
- net +5: track 517.3 -> 509.2 mm, vias 37 -> 38
- net /Channel1/VOS3: track 46.7 -> 42.8 mm
- net +8: track 243.5 -> 246.4 mm
- net Net-(U12-Pad5): track 13.5 -> 15.1 mm
- net /Channel1/#ATT1: track 43.3 -> 44.9 mm
- net Net-(U4-Pad5): track 13.7 -> 15.0 mm
- net (no net): track 0.00 -> 0.71 mm
Other:
- board size 100 x 100.2 mm -> 100 x 100 mm
