File: Frontend/frontend.sch (KiCad schematic (older format))
At the start: 15 parts, among them J1 VOCM, J2 BNC, J3 UMC, J4 UMC, J5 VOCM, J6 BNC, J7 UMC, J8 UMC, J9 PCIEx4 EDGE

Commit message: Schematic cleanup
Parts:
- removed E6, E7: 600, IPC7351-Nominal:INDC1005X60, symbol BEAD-0402
Connections:
- net SCL: now also J9.B6
- net SDA: now also J9.B5
Other:
- moved on the sheet: E1, TP10, TP8, TP9
Changed lines of the file:
@@
 encoding utf-8
 Sheet 1 6
-Title ""
-Date ""
-Rev ""
-Comp ""
+Title "OS-1 Oscilloscope Frontend - Dual Channel"
+Date "2015-05-17"
+Rev "A"
+Comp "c4757p"
 Comment1 ""
 Comment2 ""
@@
 NoConn ~ 2400 4700
 NoConn ~ 2400 4800
-Text Label 1350 4900 0    50   ~ 0
+Text Label 1650 4900 2    50   ~ 0
 #IRQ
 $Comp
 L +3.3 #PWR04
 U 1 1 5530714C
-P 1100 4600
-F 0 "#PWR04" H 1100 4650 30  0001 C CNN
-F 1 "+3.3" V 1100 4800 50  0000 C CNN
-F 2 "" H 1100 4600 60  0000 C CNN
-F 3 "" H 1100 4600 60  0000 C CNN
-	1    1100 4600
+P 1000 4800
+F 0 "#PWR04" H 1000 4850 30  0001 C CNN
+F 1 "+3.3" V 1000 5000 50  0000 C CNN
+F 2 "" H 1000 4800 60  0000 C CNN
+F 3 "" H 1000 4800 60  0000 C CNN
+	1    1000 4800
 	0    -1   -1   0
 $EndComp
@@
 	0    1    1    0
 $EndComp
-Text Label 2050 3400 0    50   ~ 0
+Text Label 1650 4400 2    50   ~ 0
 SCL
-Text Label 2050 3550 0    50   ~ 0
+Text Label 1650 4300 2    50   ~ 0
 SDA
 $Comp
@@
 L BEAD-1206 E1
 U 1 1 55451505
-P 1400 4600
-F 0 "E1" H 1400 4700 50  0000 C CNN
-F 1 "120" H 1400 4500 50  0000 C CNN
-F 2 "IPC7351-Nominal:RESC3216X60" H 1400 4600 50  0001 C CNN
-F 3 "" H 1400 4650 60  0000 C CNN
-F 4 "742792113" H 1400 4600 60  0001 C CNN "PN"
-F 5 "Wurth" H 1400 4600 60  0001 C CNN "Manuf"
-F 6 "DIST DIGIKEY 732-1622-1-ND" H 1400 4600 60  0001 C CNN "BOM"
-	1    1400 4600
+P 1300 4800
+F 0 "E1" H 1300 5000 50  0000 C CNN
+F 1 "120" H 1300 4900 50  0000 C CNN
+F 2 "IPC7351-Nominal:RESC3216X60" H 1300 4800 50  0001 C CNN
+F 3 "" H 1300 4850 60  0000 C CNN
+F 4 "742792113" H 1300 4800 60  0001 C CNN "PN"
+F 5 "Wurth" H 1300 4800 60  0001 C CNN "Manuf"
+F 6 "DIST DIGIKEY 732-1622-1-ND" H 1300 4800 60  0001 C CNN "BOM"
+	1    1300 4800
 	1    0    0    -1
 $EndComp
@@
 	2400 4000 2500 4000
 Wire Wire Line
-	2500 4000 2500 4100
+	2500 4000 2500 4050
+Wire Wire Line
+	2500 4050 2500 4100
 Wire Wire Line
 	2500 4100 2400 4100
@@
 	1850 4200 1900 4200
 Wire Wire Line
-	1650 3900 1900 3900
-Wire Wire Line
-	1850 3900 1850 4100
+	1650 3900 1750 3900
+Wire Wire Line
+	1750 3900 1850 3900
+Wire Wire Line
+	1850 3900 1900 3900
+Wire Wire Line
+	1850 3900 1850 4000
+Wire Wire Line
+	1850 4000 1850 4100
 Wire Wire Line
 	1850 4100 1900 4100
@@
 	1900 5200 1800 5200
 Wire Wire Line
-	1800 5150 1800 7300
+	1800 5150 1800 5200
+Wire Wire Line
+	1800 5200 1800 5500
+Wire Wire Line
+	1800 5500 1800 5700
+Wire Wire Line
+	1800 5700 1800 6100
+Wire Wire Line
+	1800 6100 1800 6200
+Wire Wire Line
+	1800 6200 1800 6500
+Wire Wire Line
+	1800 6500 1800 6600
+Wire Wire Line
+	1800 6600 1800 6900
+Wire Wire Line
+	1800 6900 1800 7100
+Wire Wire Line
+	1800 7100 1800 7200
+Wire Wire Line
+	1800 7200 1800 7300
 Wire Wire Line
 	1900 7200 1800 7200
@@
 	2400 5100 2500 5100
 Wire Wire Line
-	2500 5100 2500 7300
+	2500 5100 2500 5400
+Wire Wire Line
+	2500 5400 2500 5700
+Wire Wire Line
+	2500 5700 2500 6000
+Wire Wire Line
+	2500 6000 2500 6300
+Wire Wire Line
+	2500 6300 2500 6400
+Wire Wire Line
+	2500 6400 2500 6700
+Wire Wire Line
+	2500 6700 2500 6800
+Wire Wire Line
+	2500 6800 2500 7100
+Wire Wire Line
+	2500 7100 2500 7300
 Wire Wire Line
 	2500 7100 2400 7100
@@
 	900  3550 900  4300
 Wire Wire Line
-	800  4400 800  3400
-Wire Wire Line
-	3100 3400 3100 4100
+	800  4400 800  3450
+Wire Wire Line
+	3100 3450 3100 4100
 Wire Wire Line
 	3100 4100 3800 4100
 Wire Wire Line
-	1100 4600 1300 4600
-Wire Wire Line
-	1500 4600 1650 4600
-Wire Wire Line
-	1650 4600 1650 4800
-Wire Wire Line
-	1650 4800 1900 4800
+	1000 4800 1100 4800
+Wire Wire Line
+	1100 4800 1200 4800
 Wire Wire Line
 	3800 4000 3200 4000
 Wire Wire Line
-	3200 4000 3200 3250
-Wire Wire Line
-	3200 3250 600  3250
-Wire Wire Line
-	600  3250 600  4900
+	3200 4000 3200 3350
+Wire Wire Line
+	3200 3350 600  3350
+Wire Wire Line
+	600  3350 600  4900
 Wire Wire Line
 	7450 1150 7550 1150
@@
 	9150 3900 9050 3900
 Wire Wire Line
-	5100 6100 9250 6100
-Wire Wire Line
-	9250 6100 9250 2400
-Wire Wire Line
-	9250 2400 9050 2400
+	5100 6100 10100 6100
+Wire Wire Line
+	10100 6100 10100 2400
+Wire Wire Line
+	10100 2400 9050 2400
 Wire Wire Line
 	3800 3900 3400 3900
@@
 L PWR #PWR019
 U 1 1 5557EAD3
-P 1200 4550
-F 0 "#PWR019" H 1200 4550 50  0001 C CNN
-F 1 "PWR" H 1200 4550 50  0001 C CNN
-F 2 "" H 1200 4550 60  0000 C CNN
-F 3 "" H 1200 4550 60  0000 C CNN
-	1    1200 4550
+P 1100 4750
+F 0 "#PWR019" H 1100 4750 50  0001 C CNN
+F 1 "PWR" H 1100 4750 50  0001 C CNN
+F 2 "" H 1100 4750 60  0000 C CNN
+F 3 "" H 1100 4750 60  0000 C CNN
+	1    1100 4750
 	1    0    0    -1
 $EndComp
@@
 Connection ~ 1750 3900
 Wire Wire Line
-	1200 4550 1200 4600
-Connection ~ 1200 4600
+	1100 4750 1100 4800
+Connection ~ 1100 4800
 $Comp
 L PWR #PWR020
@@
 L TESTPOINT TP8
 U 1 1 5558DEAC
-P 4900 7200
-F 0 "TP8" H 5050 7350 50  0000 C CNN
-F 1 "+5" H 5050 7250 50  0000 C CNN
-F 2 "conn-test:TEST-SMD-SMALL" H 4900 7200 50  0001 C CNN
-F 3 "" H 4900 7200 50  0000 C CNN
-	1    4900 7200
+P 4000 7500
+F 0 "TP8" H 4150 7650 50  0000 C CNN
+F 1 "+5" H 4150 7550 50  0000 C CNN
+F 2 "conn-test:TEST-SMD-SMALL" H 4000 7500 50  0001 C CNN
+F 3 "" H 4000 7500 50  0000 C CNN
+	1    4000 7500
 	1    0    0    -1
 $EndComp
@@
 L +5 #PWR021
 U 1 1 5558E053
-P 4900 7200
-F 0 "#PWR021" H 4900 7250 30  0001 C CNN
-F 1 "+5" H 4900 7300 50  0000 C CNN
-F 2 "" H 4900 7200 60  0000 C CNN
-F 3 "" H 4900 7200 60  0000 C CNN
-	1    4900 7200
+P 4000 7500
+F 0 "#PWR021" H 4000 7550 30  0001 C CNN
+F 1 "+5" H 4000 7600 50  0000 C CNN
+F 2 "" H 4000 7500 60  0000 C CNN
+F 3 "" H 4000 7500 60  0000 C CNN
+	1    4000 7500
 	-1   0    0    1
 $EndComp
@@
 L TESTPOINT TP9
 U 1 1 5558E378
-P 5250 7200
-F 0 "TP9" H 5400 7350 50  0000 C CNN
-F 1 "-5" H 5400 7250 50  0000 C CNN
-F 2 "conn-test:TEST-SMD-SMALL" H 5250 7200 50  0001 C CNN
-F 3 "" H 5250 7200 50  0000 C CNN
-	1    5250 7200
+P 4350 7500
+F 0 "TP9" H 4500 7650 50  0000 C CNN
+F 1 "-5" H 4500 7550 50  0000 C CNN
+F 2 "conn-test:TEST-SMD-SMALL" H 4350 7500 50  0001 C CNN
+F 3 "" H 4350 7500 50  0000 C CNN
+	1    4350 7500
 	1    0    0    -1
 $EndComp
@@
 L -5 #PWR022
 U 1 1 5558E5C7
-P 5250 7200
-F 0 "#PWR022" H 5250 7150 30  0001 C CNN
-F 1 "-5" H 5250 7100 50  0000 C CNN
-F 2 "" H 5250 7200 60  0000 C CNN
-F 3 "" H 5250 7200 60  0000 C CNN
-	1    5250 7200
+P 4350 7500
+F 0 "#PWR022" H 4350 7450 30  0001 C CNN
+F 1 "-5" H 4350 7400 50  0000 C CNN
+F 2 "" H 4350 7500 60  0000 C CNN
+F 3 "" H 4350 7500 60  0000 C CNN
+	1    4350 7500
 	1    0    0    -1
 $EndComp
@@
 L TESTPOINT TP10
 U 1 1 5558E8F0
-P 5600 7200
-F 0 "TP10" H 5750 7350 50  0000 C CNN
-F 1 "+3.3A" H 5750 7250 50  0000 C CNN
-F 2 "conn-test:TEST-SMD-SMALL" H 5600 7200 50  0001 C CNN
-F 3 "" H 5600 7200 50  0000 C CNN
-	1    5600 7200
-	1    0    0    -1
-$EndComp
-Text GLabel 5600 7300 3    50   Output ~ 0
+P 4700 7500
+F 0 "TP10" H 4850 7650 50  0000 C CNN
+F 1 "+3.3A" H 4850 7550 50  0000 C CNN
+F 2 "conn-test:TEST-SMD-SMALL" H 4700 7500 50  0001 C CNN
+F 3 "" H 4700 7500 50  0000 C CNN
+	1    4700 7500
+	1    0    0    -1
+$EndComp
+Text GLabel 4700 7600 3    50   Output ~ 0
 +3.3A
 Wire Wire Line
-	5600 7300 5600 7200
-$Comp
-L BEAD-0402 E?
-U 1 1 555A74A2
-P 1500 3400
-AR Path="/552B011F/555A74A2" Ref="E?"  Part="1"
-AR Path="/555A74A2" Ref="E6"  Part="1"
-F 0 "E6" H 1500 3600 50  0000 C CNN
-F 1 "600" H 1500 3500 50  0000 C CNN
-F 2 "IPC7351-Nominal:INDC1005X60" H 1500 3400 50  0001 C CNN
-F 3 "" H 1500 3450 60  0000 C CNN
-F 4 "PE-0402FB601ST" H 1500 3400 60  0001 C CNN "PN"
-F 5 "Pulse" H 1500 3400 60  0001 C CNN "Manuf"
-F 6 "DIST DIGIKEY 553-2374-1-ND" H 1500 3400 60  0001 C CNN "BOM"
-	1    1500 3400
-	1    0    0    -1
-$EndComp
-$Comp
-L BEAD-0402 E?
-U 1 1 555A757C
-P 1800 3550
-AR Path="/552B011F/555A757C" Ref="E?"  Part="1"
-AR Path="/555A757C" Ref="E7"  Part="1"
-F 0 "E7" H 1800 3750 50  0000 C CNN
-F 1 "600" H 1800 3650 50  0000 C CNN
-F 2 "IPC7351-Nominal:INDC1005X60" H 1800 3550 50  0001 C CNN
-F 3 "" H 1800 3600 60  0000 C CNN
-F 4 "PE-0402FB601ST" H 1800 3550 60  0001 C CNN "PN"
-F 5 "Pulse" H 1800 3550 60  0001 C CNN "Manuf"
-F 6 "DIST DIGIKEY 553-2374-1-ND" H 1800 3550 60  0001 C CNN "BOM"
-	1    1800 3550
-	1    0    0    -1
-$EndComp
-Wire Wire Line
-	800  3400 1400 3400
-Wire Wire Line
-	1600 3400 3100 3400
-Wire Wire Line
-	3000 3550 1900 3550
-Wire Wire Line
-	1700 3550 900  3550
+	4700 7600 4700 7500
+Wire Wire Line
+	800  3450 3100 3450
+Wire Wire Line
+	900  3550 3000 3550
+Wire Wire Line
+	1900 4800 1400 4800
 $EndSCHEMATC

Commit message: Cleanup offset compensation system
Changed lines of the file:
@@
 	2400 4000 2500 4000
 Wire Wire Line
-	2500 4000 2500 4050
-Wire Wire Line
-	2500 4050 2500 4100
+	2500 4000 2500 4100
 Wire Wire Line
 	2500 4100 2400 4100
@@
 	1850 4200 1900 4200
 Wire Wire Line
-	1650 3900 1750 3900
+	1650 3900 1900 3900
 Wire Wire Line
-	1750 3900 1850 3900
-Wire Wire Line
-	1850 3900 1900 3900
-Wire Wire Line
-	1850 3900 1850 4000
-Wire Wire Line
-	1850 4000 1850 4100
+	1850 3900 1850 4100
 Wire Wire Line
 	1850 4100 1900 4100
@@
 	1900 5200 1800 5200
 Wire Wire Line
-	1800 5150 1800 5200
-Wire Wire Line
-	1800 5200 1800 5500
-Wire Wire Line
-	1800 5500 1800 5700
-Wire Wire Line
-	1800 5700 1800 6100
-Wire Wire Line
-	1800 6100 1800 6200
-Wire Wire Line
-	1800 6200 1800 6500
-Wire Wire Line
-	1800 6500 1800 6600
-Wire Wire Line
-	1800 6600 1800 6900
-Wire Wire Line
-	1800 6900 1800 7100
-Wire Wire Line
-	1800 7100 1800 7200
-Wire Wire Line
-	1800 7200 1800 7300
+	1800 5150 1800 7300
 Wire Wire Line
 	1900 7200 1800 7200
@@
 	2400 5100 2500 5100
 Wire Wire Line
-	2500 5100 2500 5400
-Wire Wire Line
-	2500 5400 2500 5700
-Wire Wire Line
-	2500 5700 2500 6000
-Wire Wire Line
-	2500 6000 2500 6300
-Wire Wire Line
-	2500 6300 2500 6400
-Wire Wire Line
-	2500 6400 2500 6700
-Wire Wire Line
-	2500 6700 2500 6800
-Wire Wire Line
-	2500 6800 2500 7100
-Wire Wire Line
-	2500 7100 2500 7300
+	2500 5100 2500 7300
 Wire Wire Line
 	2500 7100 2400 7100
@@
 	3100 4100 3800 4100
 Wire Wire Line
-	1000 4800 1100 4800
-Wire Wire Line
-	1100 4800 1200 4800
+	1000 4800 1200 4800
 Wire Wire Line
 	3800 4000 3200 4000

Commit message: Even more layout tweaks
Parts:
- E1: BOM DIST DIGIKEY 732-1622-1-ND -> BEAD SMD 120 1A [1206]
- J3, J4, J7, J8: BOM (none) -> DIST DIGIKEY WM5587CT-ND; Manuf (none) -> Molex; PN (none) -> 0734120110
Connections:
- net 3V3SB: now reaches E1.2, J9.B10
Other:
- note added: "The system design requires the card-identifying I2C device to\nbe powered from 3V3SB. On this card, the main microcontroller\nperforms this function. Because the load on the 3V3 rail here\nis so small, we're using 3V3SB as the main 3V3 rail for simplicity.\n\nUnused edge contacts A9,A10,B8,B9 are the master 3V3 rail."
Changed lines of the file:
@@
 F0 "Channel1" 60
 F1 "Channel.sch" 60
-F2 "VOS1" I L 7900 1600 60
-F3 "VOCM" I L 7900 1500 60
-F4 "VO_P" O R 9050 1300 60
-F5 "VO_N" O R 9050 1400 60
-F6 "VOS2" I L 7900 1700 60
-F7 "INPUT" I L 7900 1300 60
-F8 "VOS3" I L 7900 1800 60
-F9 "#TERM" I L 7900 1900 60
-F10 "#ATT1" I L 7900 2000 60
+F2 "VOS1" I L 7900 1600 50
+F3 "VOCM" I L 7900 1500 50
+F4 "VO_P" O R 9050 1300 50
+F5 "VO_N" O R 9050 1400 50
+F6 "VOS2" I L 7900 1700 50
+F7 "INPUT" I L 7900 1300 50
+F8 "VOS3" I L 7900 1800 50
+F9 "#TERM" I L 7900 1900 50
+F10 "#ATT1" I L 7900 2000 50
 F11 "#DC" I L 7900 2100 50
 F12 "ATT2" I L 7900 2200 50
@@
 F0 "Channel2" 60
 F1 "Channel.sch" 60
-F2 "VOS1" I L 7900 3100 60
-F3 "VOCM" I L 7900 3000 60
-F4 "VO_P" O R 9050 2800 60
-F5 "VO_N" O R 9050 2900 60
-F6 "VOS2" I L 7900 3200 60
-F7 "INPUT" I L 7900 2800 60
-F8 "VOS3" I L 7900 3300 60
-F9 "#TERM" I L 7900 3400 60
-F10 "#ATT1" I L 7900 3500 60
+F2 "VOS1" I L 7900 3100 50
+F3 "VOCM" I L 7900 3000 50
+F4 "VO_P" O R 9050 2800 50
+F5 "VO_N" O R 9050 2900 50
+F6 "VOS2" I L 7900 3200 50
+F7 "INPUT" I L 7900 2800 50
+F8 "VOS3" I L 7900 3300 50
+F9 "#TERM" I L 7900 3400 50
+F10 "#ATT1" I L 7900 3500 50
 F11 "#DC" I L 7900 3600 50
 F12 "ATT2" I L 7900 3700 50
@@
 $EndSheet
 $Sheet
-S 1700 1600 1000 1000
+S 1700 1100 1000 1000
 U 552F27A6
 F0 "Power" 50
 F1 "Power.sch" 50
-F2 "TEMP_VRELAY" O R 2700 1700 50
-F3 "TEMP_V5" O R 2700 1800 50
+F2 "TEMP_VRELAY" O R 2700 1200 50
+F3 "TEMP_V5" O R 2700 1300 50
 $EndSheet
 $Comp
@@
 U 1 1 553062B4
 P 2150 3900
-F 0 "J9" H 2150 4150 50  0000 C CNN
-F 1 "PCIEx4 EDGE" H 2150 4050 50  0000 C CNN
+F 0 "J9" H 2150 4100 50  0000 C CNN
+F 1 "PCIEx4 EDGE" H 2150 4000 50  0000 C CNN
 F 2 "conn-fci:CONN-10018784-10201TLF-PCIEx4-FCI" H 2150 4000 50  0001 C CNN
 F 3 "" H 2125 3900 50  0000 C CNN
@@
 F 4 "742792113" H 1300 4800 60  0001 C CNN "PN"
 F 5 "Wurth" H 1300 4800 60  0001 C CNN "Manuf"
-F 6 "DIST DIGIKEY 732-1622-1-ND" H 1300 4800 60  0001 C CNN "BOM"
+F 6 "BEAD SMD 120 1A [1206]" H 1300 4800 60  0001 C CNN "BOM"
 	1    1300 4800
 	1    0    0    -1
@@
 F 2 "conn-molex:CONN-MOLEX-0734120110" H 9800 1300 50  0001 C CNN
 F 3 "" H 9800 1300 50  0000 C CNN
+F 4 "0734120110" H 9800 1300 60  0001 C CNN "PN"
+F 5 "Molex" H 9800 1300 60  0001 C CNN "Manuf"
+F 6 "DIST DIGIKEY WM5587CT-ND" H 9800 1300 60  0001 C CNN "BOM"
 	1    9800 1300
 	-1   0    0    -1
@@
 F 2 "conn-molex:CONN-MOLEX-0734120110" H 9800 1750 50  0001 C CNN
 F 3 "" H 9800 1750 50  0000 C CNN
+F 4 "0734120110" H 9800 1750 60  0001 C CNN "PN"
+F 5 "Molex" H 9800 1750 60  0001 C CNN "Manuf"
+F 6 "DIST DIGIKEY WM5587CT-ND" H 9800 1750 60  0001 C CNN "BOM"
 	1    9800 1750
 	-1   0    0    -1
@@
 F 2 "conn-molex:CONN-MOLEX-0734120110" H 9800 2800 50  0001 C CNN
 F 3 "" H 9800 2800 50  0000 C CNN
+F 4 "0734120110" H 9800 2800 60  0001 C CNN "PN"
+F 5 "Molex" H 9800 2800 60  0001 C CNN "Manuf"
+F 6 "DIST DIGIKEY WM5587CT-ND" H 9800 2800 60  0001 C CNN "BOM"
 	1    9800 2800
 	-1   0    0    -1
@@
 F 2 "conn-molex:CONN-MOLEX-0734120110" H 9800 3250 50  0001 C CNN
 F 3 "" H 9800 3250 50  0000 C CNN
+F 4 "0734120110" H 9800 3250 60  0001 C CNN "PN"
+F 5 "Molex" H 9800 3250 60  0001 C CNN "Manuf"
+F 6 "DIST DIGIKEY WM5587CT-ND" H 9800 3250 60  0001 C CNN "BOM"
 	1    9800 3250
 	-1   0    0    -1
@@
 	3800 3900 3400 3900
 Wire Wire Line
-	3400 3900 3400 1800
-Wire Wire Line
-	3400 1800 2700 1800
-Wire Wire Line
-	2700 1700 3500 1700
-Wire Wire Line
-	3500 1700 3500 3800
+	3400 3900 3400 1300
+Wire Wire Line
+	3400 1300 2700 1300
+Wire Wire Line
+	2700 1200 3500 1200
+Wire Wire Line
+	3500 1200 3500 3800
 Wire Wire Line
 	3500 3800 3800 3800
@@
 Wire Wire Line
 	1900 4800 1400 4800
+Text Label 1500 4800 0    50   ~ 0
+3V3SB
+Text Notes 600  3200 0    50   ~ 0
+The system design requires the card-identifying I2C device to\nbe powered from 3V3SB. On this card, the main microcontroller\nperforms this function. Because the load on the 3V3 rail here\nis so small, we're using 3V3SB as the main 3V3 rail for simplicity.\n\nUnused edge contacts A9,A10,B8,B9 are the master 3V3 rail.
 $EndSCHEMATC
